File: kicad/hierophone.kicad_pcb (KiCad board)
At the start: 2 copper layers, 220 x 130 mm, 171 parts, among them J1 AudioJack2_SwitchT, J10 Conn_01x02, J13 AudioJack2_SwitchT, J2 AudioJack2_SwitchT, J3 Conn_01x03_Pin, J4 AudioJack2_SwitchT, J5 AudioJack2_SwitchT, J6 AudioJack2_SwitchT, J7 AudioJack2_SwitchT, J8 Conn_01x02, J9 Conn_01x02, Q1 2N3904, Q2 2N3906, Q3 2N3906, SW1 SW_SPDT, SW3 SW_SPDT, U1 TL074, U10 TL072, U12 TL072, U13 TL072, U2 LM13700, U3 LM13700, U4 TL072, U5 TL072, U6 LM386, U7 NE5534, U8 TL072, U9 ICL7660

Commit message: Regenerating gerbers
Parts:
- U6: value LM386 -> LM386N-4
Changed lines of the file:
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@@
 			)
 		)
-		(property "Value" "LM386"
+		(property "Value" "LM386N-4"
 			(at 3.8 8.118 0)
 			(layer "F.Fab")
@@
 		(tags "connector Molex KK-254 side entry")
 		(property "Reference" "J9"
-			(at 1.27 -2.54 0)
+			(at 5.207 0 0)
 			(layer "F.SilkS")
 			(effects
@@
 		)
 		(fp_text user "${REFERENCE}"
-			(at 1.27 -2.54 0)
+			(at 5.207 0 0)
 			(layer "F.Fab")
 			(effects
